Commit message: added two new pkgs 1 for object detection with yolov8 and 2 for the simulation of the human within gazebo environment

File: src/amr_description/urdf/amr.urdf.xacro (robot description, xacro)
@@ -191,4 +191,35 @@
     </collision>
   </link>
+  <link name='camera_link'>
+    <pose>0 0 0 0 0 0</pose>
+    <collision name='collision'>
+      <origin xyz="0 0 0" rpy="0 0 0"/>
+      <geometry>
+        <box size=".02 .02 .02"/>
+      </geometry>
+    </collision>
+    <visual name='camera_link_visual'>
+      <origin xyz="0 0 0" rpy="0 0 0"/>
+      <geometry>
+        <box size=".02 .02 .02"/>
+      </geometry>
+    </visual>
+  </link>
+  <joint type="fixed" name="camera_joint">
+    <origin xyz="0.05 0 -0.006" rpy="0 0 0"/>
+    <child link="camera_link"/>
+    <parent link="robot_base"/>
+    <axis xyz="0 1 0" />
+  </joint>
+  <gazebo reference="camera_link">
+    <material>Gazebo/Red</material>
+  </gazebo>
+  <joint type="fixed" name="camera_optical_joint">
+    <origin xyz="0 0 0" rpy="-1.5707 0 -1.5707"/>
+    <child link="camera_link_optical"/>
+    <parent link="camera_link"/>
+  </joint>
+  <link name="camera_link_optical">
+  </link>
   <joint name="lidar_joint" type="fixed">
     <parent link="robot_base"/>

File: src/amr_description/urdf/amr_gazebo.xacro (robot description, xacro)
@@ -124,3 +124,33 @@
         </sensor>
     </gazebo>
+    <gazebo reference="camera_link">
+        <sensor name="camera" type="camera">
+        <camera>
+            <horizontal_fov>1.3962634</horizontal_fov>
+            <image>
+            <width>640</width>
+            <height>480</height>
+            <format>R8G8B8</format>
+            </image>
+            <clip>
+            <near>0.1</near>
+            <far>15</far>
+            </clip>
+            <noise>
+            <type>gaussian</type>
+            <!-- Noise is sampled independently per pixel on each frame.
+                That pixel's noise value is added to each of its color
+                channels, which at that point lie in the range [0,1]. -->
+            <mean>0.0</mean>
+            <stddev>0.007</stddev>
+            </noise>
+            <optical_frame_id>camera_link_optical</optical_frame_id>
+            <camera_info_topic>camera/camera_info</camera_info_topic>
+        </camera>
+        <always_on>1</always_on>
+        <update_rate>20</update_rate>
+        <visualize>true</visualize>
+        <topic>camera/image</topic>
+        </sensor>
+    </gazebo>
 </robot>

Commit message: added new package for training deep reinforcement learning for autonomous navigation

File: src/amr_description/urdf/amr.urdf.xacro (robot description, xacro)
@@ -140,5 +140,5 @@
     <axis xyz="0 0 0" />
   </joint>
-  <link name="imu_link">
+  <!--link name="imu_link">
     <inertial>
       <origin xyz="-0.00552433659106688 0.000168210391520346 0.000514000497342681" rpy="0 0 0" />
@@ -169,5 +169,5 @@
     <child link="imu_link" />
     <axis xyz="0 0 0" />
-  </joint>
+  </joint-->
   <link name="lidar_link">
     <inertial>
@@ -191,5 +191,5 @@
     </collision>
   </link>
-  <link name='camera_link'>
+  <!--link name='camera_link'>
     <pose>0 0 0 0 0 0</pose>
     <collision name='collision'>
@@ -221,5 +221,5 @@
   </joint>
   <link name="camera_link_optical">
-  </link>
+  </link-->
   <joint name="lidar_joint" type="fixed">
     <parent link="robot_base"/>

File: src/amr_description/urdf/amr_gazebo.xacro (robot description, xacro)
@@ -44,6 +44,13 @@
         <render_engine>ogre2</render_engine>
       </plugin>
+      <plugin
+            filename="gz-sim-pose-publisher-system"
+            name="gz::sim::systems::PosePublisher">
+            <publish_link_pose>true</publish_link_pose>
+            <use_pose_vector_msg>true</use_pose_vector_msg>
+            <publish_nested_model_pose>true</publish_nested_model_pose>
+      </plugin>
     </gazebo>
-    <gazebo reference="imu_link">
+    <!--gazebo reference="imu_link">
         <sensor name="imu" type="imu">
             <always_on>true</always_on>
@@ -94,5 +101,5 @@
             </imu>
         </sensor>
-    </gazebo>
+    </gazebo-->
     <gazebo reference="lidar_link">
         <sensor name="lidar" type="gpu_lidar">
@@ -112,6 +119,6 @@
                 </scan>
                 <range>
-                    <min>0.100000</min>
-                    <max>5.5</max>
+                    <min>0.0500000</min>
+                    <max>10</max>
                     <resolution>0.02</resolution>
                 </range>
@@ -124,5 +131,5 @@
         </sensor>
     </gazebo>
-    <gazebo reference="camera_link">
+    <!--gazebo reference="camera_link">
         <sensor name="camera" type="camera">
         <camera>
@@ -139,7 +146,7 @@
             <noise>
             <type>gaussian</type>
-            <!-- Noise is sampled independently per pixel on each frame.
+            < Noise is sampled independently per pixel on each frame.
                 That pixel's noise value is added to each of its color
-                channels, which at that point lie in the range [0,1]. -->
+                channels, which at that point lie in the range [0,1]. >
             <mean>0.0</mean>
             <stddev>0.007</stddev>
@@ -153,4 +160,4 @@
         <topic>camera/image</topic>
         </sensor>
-    </gazebo>
+    </gazebo-->
 </robot>
